File: cad/opsis.kicad_sch (KiCad schematic)
At the start: 11 parts, among them J101 Conn_01x02, J102 Conn_01x02, J103 REGULATOR, J104 Conn_01x02, J105 Conn_01x02, J106 Conn_01x04_MountingPin, J107 Conn_01x02, J108 USB_A

Commit message: initial rev made
Parts:
- removed H101, H102, H103: MountingHole, MountingHole:MountingHole_3.2mm_M3_Pad, symbol Mechanical:MountingHole
- added J101: Conn_01x02, Connector_Phoenix_MC:PhoenixContact_MC_1,5_2-G-3.81_1x02_P3.81mm_Horizontal, symbol Connector_Generic:Conn_01x02
- added JP101: Jumper_2_Open, Jumper:SolderJumper-2_P1.3mm_Open_RoundedPad1.0x1.5mm, symbol Jumper:Jumper_2_Open
- renumbered J101 to J102, J102 to J103, J103 to J104, J106 to J105, J104 to J106, J105 to J107, J107 to J108, J108 to J109
Connections:
- net GND: now also J105.MP (MountPin), J106.1 (Pin_1), J107.1 (Pin_1), J101.2 (Pin_2); no longer J106.2 (Pin_2), J107.2 (Pin_2)
- net at J102.1 (Pin_1), J103.1 (Pin_1), J104.1 (Pin_1): now also J105.1 (Pin_1), J101.1 (Pin_1); no longer J105.4 (Pin_4)
- net at J108.2 (Pin_2), J109.1 (VBUS): now also J105.4 (Pin_4), JP101.2 (B); no longer J105.1 (Pin_1)
- new net: J104.4 (Pin_4), J106.2 (Pin_2), J107.2 (Pin_2), JP101.1 (A)
Other:
- moved on the sheet: J105, J106, J107
